File: KiCad/CABR_Schematic.kicad_pcb (KiCad board)
At the start: 2 copper layers, 23.5 x 59.1 mm, 19 parts, among them J1 Screw_Terminal_01x02, J2 0.1" Header, J3 Program Header, J4 MicroSwitch, J5 Screw_Terminal_01x02, Q1 PBSS4250X, U1 AZ1117-5.0, U2 ATtiny85-20SU

Commit message: updated PCB and gerber files
Parts:
- added REF**: OSHW-Logo2_7.3x6mm_SilkScreen, Symbol:OSHW-Logo2_7.3x6mm_SilkScreen, F.Cu at (142.5, 72.6)
- moved C2 10.8 mm to (155.2, 97.8), turned to 270 degrees
- moved C1 8.53 mm to (143.3, 99.6), turned to 90 degrees
- moved D2 7.38 mm to (152.7, 70.6), turned to 180 degrees
Routing:
- net GND: track 85.5 -> 112.9 mm, vias 5 -> 6
- net Net-(C1-Pad1): track 57.7 -> 63.1 mm, vias 3 -> 2
- net Net-(C2-Pad1): track 61.2 -> 57.5 mm, vias 4 -> 2
- net Net-(D2-Pad2): track 16.4 -> 19.6 mm
