File: KiCad/CABR_Schematic.kicad_pcb (KiCad board)
At the start: 2 copper layers, 23.5 x 54.6 mm, 20 parts, among them J1 Screw_Terminal_01x02, J2 0.1" Header, J3 Program Header, J4 MicroSwitch, J5 Screw_Terminal_01x02, Q1 PBSS4250X, U1 AZ1117-5.0, U2 ATtiny85-20SU

Commit message: updated design and fixed output pins
Parts:
- removed C3: 0.1uF, Capacitor_SMD:C_0805_2012Metric
- J1, J5: value Screw_Terminal_01x02 -> XT60
Connections:
- U2 pad 8: Net-(C3-Pad1) -> Net-(C2-Pad1)
Routing:
- net Net-(C3-Pad1): track 3.30 -> 0.00 mm
- net Net-(C2-Pad1): track 55.7 -> 56.2 mm, vias 2 -> 1
Other:
- board text added: "chand1012"

Commit message: more board updates
Parts:
- added C3: 0.1uF, Capacitor_SMD:C_0805_2012Metric, F.Cu at (156.0, 80.5)
- moved R2 3.11 mm to (156.0, 83.6), turned to 0 degrees
- moved R1 1.27 mm to (155.9, 90.2), turned to 180 degrees
- moved D1 1.02 mm to (143.3, 91.4)
- moved R5 0.48 mm to (156.0, 85.9), turned to 180 degrees
Routing:
- net Net-(J2-Pad2): track 23.2 -> 19.3 mm
- net Net-(C2-Pad1): track 56.2 -> 52.4 mm
- net Net-(J2-Pad3): track 25.9 -> 23.4 mm
- net GND: track 118.2 -> 116.4 mm
- net Net-(J4-Pad2): track 27.9 -> 26.2 mm

Commit message: more modifications
Parts:
- moved R6 5.01 mm to (149.9, 77.2), turned to 270 degrees
- moved Q1 2.04 mm to (154.4, 75.7), turned to 90 degrees
- moved J3 0.18 mm to (151.9, 88.1)
Connections:
- J3 pad 2: Net-(J2-Pad3) -> Net-(C2-Pad1)
- J3 pad 3: Net-(J3-Pad3) -> Net-(J2-Pad3)
- J3 pad 4: Net-(C2-Pad1) -> Net-(J3-Pad4)
- Q1 pad 1: GND -> Net-(Q1-Pad1)
- Q1 pad 3: Net-(Q1-Pad3) -> GND
- R5 pad 2: Net-(J3-Pad5) -> Net-(J3-Pad4)
- R6 pad 1: Net-(Q1-Pad3) -> Net-(Q1-Pad1)
- R6 pad 2: Net-(J3-Pad5) -> Net-(J3-Pad4)
- U2 pad 1: Net-(J3-Pad3) -> Net-(J3-Pad5)
- U2 pad 5: Net-(J3-Pad5) -> Net-(J3-Pad4)
Routing:
- net GND: track 116.4 -> 82.4 mm, vias 2 -> 1
- net Net-(J3-Pad4): track 0.00 -> 20.2 mm, vias 0 -> 2
- net Net-(J3-Pad5): track 27.8 -> 9.02 mm, vias 1 -> 0
- net Net-(J3-Pad3): track 10.1 -> 0.00 mm, vias 1 -> 0
- net Net-(Q1-Pad3): track 5.86 -> 0.00 mm
- net Net-(C1-Pad1): track 61.5 -> 66.9 mm, vias 1 -> 0
- net Net-(C2-Pad1): track 52.4 -> 47.9 mm, vias 1 -> 3
- net Net-(J2-Pad2): track 19.3 -> 23.0 mm
- net Net-(Q1-Pad1): track 0.00 -> 3.44 mm
- net Net-(J2-Pad3): track 23.4 -> 25.1 mm
- net Net-(D2-Pad2): track 18.9 -> 17.3 mm
Other:
- board text added: "Rev B"

Commit message: more fixes
Parts:
- removed REF**: OSHW-Logo2_7.3x6mm_SilkScreen, Symbol:OSHW-Logo2_7.3x6mm_SilkScreen
- Q1: value PBSS4250X -> FQP30N06L; footprint Package_TO_SOT_SMD:SOT-89-3 -> Package_TO_SOT_THT:TO-220-3_Vertical
- moved Q1 13.8 mm to (140.9, 73.2), turned to 0 degrees
Connections:
- Q1 pad 2: Net-(D2-Pad2) -> GND
- Q1 pad 3: GND -> Net-(D2-Pad2)
Routing:
- net GND: track 82.4 -> 104.4 mm, vias 1 -> 2
- net Net-(Q1-Pad1): track 3.44 -> 10.3 mm
- net Net-(C2-Pad1): track 47.9 -> 54.2 mm
- net Net-(D2-Pad2): track 17.3 -> 16.3 mm

Commit message: more updates
Parts:
- moved R6 1.14 mm to (149.4, 76.2), turned to 90 degrees
- moved Q1 0.72 mm to (140.5, 72.6)
Connections:
- R6 pad 1: Net-(Q1-Pad1) -> Net-(J3-Pad4)
- R6 pad 2: Net-(J3-Pad4) -> Net-(Q1-Pad1)
Routing:
- net Net-(D2-Pad2): track 16.3 -> 14.4 mm
- net Net-(J3-Pad4): track 20.2 -> 21.4 mm
Other:
- board text added: "Female"
- board text added: "Male"
