File: KiCad/CABR_Schematic.kicad_pcb (KiCad board)
At the start: 2 copper layers, 23.5 x 54.6 mm, 19 parts, among them J1 XT60, J2 0.1" Header, J3 Program Header, J4 MicroSwitch, J5 XT60, Q1 FQP30N06L, U1 AZ1117-5.0, U2 ATtiny85-20SU

Commit message: Update CABR_Schematic.kicad_pcb
Routing:
- net GND: track 104.2 -> 96.8 mm
- net Net-(J3-Pad4): track 21.4 -> 27.6 mm, vias 2 -> 1
- net Net-(C2-Pad1): track 54.2 -> 57.5 mm, vias 3 -> 1
- net Net-(J2-Pad3): track 25.1 -> 22.1 mm
- net Net-(J2-Pad2): track 23.0 -> 22.2 mm
- net Net-(J3-Pad5): track 9.02 -> 8.31 mm
- net Net-(Q1-Pad1): track 10.0 -> 10.6 mm
